File: hub75_extension/hub75_extension.kicad_pcb (KiCad board)
At the start: 2 copper layers, 81.3 x 61 mm, 40 parts, among them J1 Screw_Terminal_01x02, J2 Screw_Terminal_01x02, J3 Barrel_Jack_Switch, J4 Screw_Terminal_01x02, J5 Screw_Terminal_01x02, J6 Barrel_Jack_Switch, J7 Screw_Terminal_01x02, J8 Screw_Terminal_01x02, J9 USB_B_Micro, U1 74HC595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

Commit message: Update HUB75 board with new netlist
Parts:
- removed J_FOUND1: Found_LED_panel, Connector_IDC:IDC-Header_2x08_P2.54mm_Vertical
- added J_HUB12_1: HUB12, Connector_PinSocket_2.54mm:PinSocket_2x08_P2.54mm_Vertical, B.Cu at (86.4, 91.4)
- added J_IN1: HUB75, Connector_IDC:IDC-Header_2x08_P2.54mm_Vertical, F.Cu at (76.2, 91.4)
- J_DS1: footprint Connector_PinHeader_2.54mm:PinHeader_2x09_P2.54mm_Vertical -> ds_card_extender:IDC-Header_2x09_P2.54mm_Vertical
- J_PANEL1: footprint Connector_IDC:IDC-Header_2x08_P2.54mm_Vertical -> Connector_PinSocket_2.54mm:PinSocket_2x08_P2.54mm_Vertical; moved to B.Cu
- turned J_PANEL1 to 180 degrees
- renumbered J_CHAIN1 to J_OUT1
Routing:
- net /C: track 81.0 -> 91.7 mm
