File: hub75_extension/hub75.sch (KiCad schematic (older format))
At the start: 23 parts

Commit message: Yeah, just renumber the entire thing...
Parts:
- renumbered JP4 to JP501, JP5 to JP502, JP6 to JP503, JP15 to JP504, JP16 to JP505, JP17 to JP506, JP18 to JP507, JP19 to JP508, JP20 to JP509, JP21 to JP510, JP23 to JP511, JP24 to JP512, JP25 to JP513, JP26 to JP514, JP27 to JP515, JP28 to JP516, JP30 to JP517
Changed lines of the file:
@@
 P 4800 2250
 AR Path="/60AB65DD" Ref="#PWR?"  Part="1"
-AR Path="/60A8CB6A/60AB65DD" Ref="#PWR04"  Part="1"
-F 0 "#PWR04" H 4800 2000 50  0001 C CNN
+AR Path="/60A8CB6A/60AB65DD" Ref="#PWR0502"  Part="1"
+F 0 "#PWR0502" H 4800 2000 50  0001 C CNN
 F 1 "GND" H 4805 2077 50  0000 C CNN
 F 2 "" H 4800 2250 50  0001 C CNN
@@
 P 6850 3750
 AR Path="/60AB6614" Ref="#PWR?"  Part="1"
-AR Path="/60A8CB6A/60AB6614" Ref="#PWR05"  Part="1"
-F 0 "#PWR05" H 6850 3500 50  0001 C CNN
+AR Path="/60A8CB6A/60AB6614" Ref="#PWR0503"  Part="1"
+F 0 "#PWR0503" H 6850 3500 50  0001 C CNN
 F 1 "GND" H 6855 3577 50  0000 C CNN
 F 2 "" H 6850 3750 50  0001 C CNN
@@
 P 9250 2200
 AR Path="/60AB663E" Ref="#PWR?"  Part="1"
-AR Path="/60A8CB6A/60AB663E" Ref="#PWR041"  Part="1"
-F 0 "#PWR041" H 9250 1950 50  0001 C CNN
+AR Path="/60A8CB6A/60AB663E" Ref="#PWR0506"  Part="1"
+F 0 "#PWR0506" H 9250 1950 50  0001 C CNN
 F 1 "GND" H 9255 2027 50  0000 C CNN
 F 2 "" H 9250 2200 50  0001 C CNN
@@
 P 9250 3750
 AR Path="/60AB6660" Ref="#PWR?"  Part="1"
-AR Path="/60A8CB6A/60AB6660" Ref="#PWR042"  Part="1"
-F 0 "#PWR042" H 9250 3500 50  0001 C CNN
+AR Path="/60A8CB6A/60AB6660" Ref="#PWR0507"  Part="1"
+F 0 "#PWR0507" H 9250 3500 50  0001 C CNN
 F 1 "GND" H 9255 3577 50  0000 C CNN
 F 2 "" H 9250 3750 50  0001 C CNN
@@
 P 9250 5150
 AR Path="/60AB6680" Ref="#PWR?"  Part="1"
-AR Path="/60A8CB6A/60AB6680" Ref="#PWR043"  Part="1"
-F 0 "#PWR043" H 9250 4900 50  0001 C CNN
+AR Path="/60A8CB6A/60AB6680" Ref="#PWR0508"  Part="1"
+F 0 "#PWR0508" H 9250 4900 50  0001 C CNN
 F 1 "GND" H 9255 4977 50  0000 C CNN
 F 2 "" H 9250 5150 50  0001 C CNN
@@
 P 6850 5150
 AR Path="/60AB66A5" Ref="#PWR?"  Part="1"
-AR Path="/60A8CB6A/60AB66A5" Ref="#PWR06"  Part="1"
-F 0 "#PWR06" H 6850 4900 50  0001 C CNN
+AR Path="/60A8CB6A/60AB66A5" Ref="#PWR0504"  Part="1"
+F 0 "#PWR0504" H 6850 4900 50  0001 C CNN
 F 1 "GND" H 6855 4977 50  0000 C CNN
 F 2 "" H 6850 5150 50  0001 C CNN
@@
 P 7200 4550
 AR Path="/60AB66C5" Ref="JP?"  Part="1"
-AR Path="/60A8CB6A/60AB66C5" Ref="JP27"  Part="1"
-F 0 "JP27" H 7400 4600 50  0000 C CNN
+AR Path="/60A8CB6A/60AB66C5" Ref="JP515"  Part="1"
+F 0 "JP515" H 7400 4600 50  0000 C CNN
 F 1 "SolderJumper_2_Bridged" H 7200 4664 50  0001 C CNN
 F 2 "Jumper:SolderJumper-2_P1.3mm_Bridged2Bar_RoundedPad1.0x1.5mm" H 7200 4550 50  0001 C CNN
@@
 P 7200 4650
 AR Path="/60AB66CB" Ref="JP?"  Part="1"
-AR Path="/60A8CB6A/60AB66CB" Ref="JP28"  Part="1"
-F 0 "JP28" H 7400 4700 50  0000 C CNN
+AR Path="/60A8CB6A/60AB66CB" Ref="JP516"  Part="1"
+F 0 "JP516" H 7400 4700 50  0000 C CNN
 F 1 "SolderJumper_2_Bridged" H 7200 4764 50  0001 C CNN
 F 2 "Jumper:SolderJumper-2_P1.3mm_Bridged2Bar_RoundedPad1.0x1.5mm" H 7200 4650 50  0001 C CNN
@@
 P 7000 4250
 AR Path="/60AB66D1" Ref="#PWR?"  Part="1"
-AR Path="/60A8CB6A/60AB66D1" Ref="#PWR07"  Part="1"
-F 0 "#PWR07" H 7000 4100 50  0001 C CNN
+AR Path="/60A8CB6A/60AB66D1" Ref="#PWR0505"  Part="1"
+F 0 "#PWR0505" H 7000 4100 50  0001 C CNN
 F 1 "+5V" H 7015 4423 50  0000 C CNN
 F 2 "" H 7000 4250 50  0001 C CNN
@@
 P 4800 4550
 AR Path="/60AB66DD" Ref="JP?"  Part="1"
-AR Path="/60A8CB6A/60AB66DD" Ref="JP24"  Part="1"
-F 0 "JP24" H 5000 4600 50  0000 C CNN
+AR Path="/60A8CB6A/60AB66DD" Ref="JP512"  Part="1"
+F 0 "JP512" H 5000 4600 50  0000 C CNN
 F 1 "SolderJumper_2_Bridged" H 4800 4664 50  0001 C CNN
 F 2 "Jumper:SolderJumper-2_P1.3mm_Bridged2Bar_RoundedPad1.0x1.5mm" H 4800 4550 50  0001 C CNN
@@
 P 4800 4650
 AR Path="/60AB66E3" Ref="JP?"  Part="1"
-AR Path="/60A8CB6A/60AB66E3" Ref="JP25"  Part="1"
-F 0 "JP25" H 5000 4700 50  0000 C CNN
+AR Path="/60A8CB6A/60AB66E3" Ref="JP513"  Part="1"
+F 0 "JP513" H 5000 4700 50  0000 C CNN
 F 1 "SolderJumper_2_Bridged" H 4800 4764 50  0001 C CNN
 F 2 "Jumper:SolderJumper-2_P1.3mm_Bridged2Bar_RoundedPad1.0x1.5mm" H 4800 4650 50  0001 C CNN
@@
 P 4600 4250
 AR Path="/60AB66E9" Ref="#PWR?"  Part="1"
-AR Path="/60A8CB6A/60AB66E9" Ref="#PWR03"  Part="1"
-F 0 "#PWR03" H 4600 4100 50  0001 C CNN
+AR Path="/60A8CB6A/60AB66E9" Ref="#PWR0501"  Part="1"
+F 0 "#PWR0501" H 4600 4100 50  0001 C CNN
 F 1 "+5V" H 4615 4423 50  0000 C CNN
 F 2 "" H 4600 4250 50  0001 C CNN
@@
 P 9000 4550
 AR Path="/60AB66F4" Ref="JP?"  Part="1"
-AR Path="/60A8CB6A/60AB66F4" Ref="JP30"  Part="1"
-F 0 "JP30" H 8800 4600 50  0000 C CNN
+AR Path="/60A8CB6A/60AB66F4" Ref="JP517"  Part="1"
+F 0 "JP517" H 8800 4600 50  0000 C CNN
 F 1 "SolderJumper_2_Bridged" H 9000 4664 50  0001 C CNN
 F 2 "Jumper:SolderJumper-2_P1.3mm_Bridged2Bar_RoundedPad1.0x1.5mm" H 9000 4550 50  0001 C CNN
@@
 P 6600 4550
 AR Path="/60AB66FA" Ref="JP?"  Part="1"
-AR Path="/60A8CB6A/60AB66FA" Ref="JP26"  Part="1"
-F 0 "JP26" H 6400 4600 50  0000 C CNN
+AR Path="/60A8CB6A/60AB66FA" Ref="JP514"  Part="1"
+F 0 "JP514" H 6400 4600 50  0000 C CNN
 F 1 "SolderJumper_2_Bridged" H 6600 4664 50  0001 C CNN
 F 2 "Jumper:SolderJumper-2_P1.3mm_Bridged2Bar_RoundedPad1.0x1.5mm" H 6600 4550 50  0001 C CNN
@@
 P 3400 1050
 AR Path="/60AC30F2" Ref="JP?"  Part="1"
-AR Path="/60A8CB6A/60AC30F2" Ref="JP4"  Part="1"
-F 0 "JP4" H 3400 1254 50  0000 C CNN
+AR Path="/60A8CB6A/60AC30F2" Ref="JP501"  Part="1"
+F 0 "JP501" H 3400 1254 50  0000 C CNN
 F 1 "Jumper_3_Bridged12" H 3400 1163 50  0000 C CNN
 F 2 "Connector_PinHeader_2.54mm:PinHeader_1x03_P2.54mm_Vertical" H 3400 1050 50  0001 C CNN
@@
 P 3400 1600
 AR Path="/60AC30FC" Ref="JP?"  Part="1"
-AR Path="/60A8CB6A/60AC30FC" Ref="JP5"  Part="1"
-F 0 "JP5" H 3400 1804 50  0000 C CNN
+AR Path="/60A8CB6A/60AC30FC" Ref="JP502"  Part="1"
+F 0 "JP502" H 3400 1804 50  0000 C CNN
 F 1 "Jumper_3_Bridged12" H 3400 1713 50  0000 C CNN
 F 2 "Connector_PinHeader_2.54mm:PinHeader_1x03_P2.54mm_Vertical" H 3400 1600 50  0001 C CNN
@@
 P 3400 2150
 AR Path="/60AC3106" Ref="JP?"  Part="1"
-AR Path="/60A8CB6A/60AC3106" Ref="JP6"  Part="1"
-F 0 "JP6" H 3400 2354 50  0000 C CNN
+AR Path="/60A8CB6A/60AC3106" Ref="JP503"  Part="1"
+F 0 "JP503" H 3400 2354 50  0000 C CNN
 F 1 "Jumper_3_Bridged12" H 3400 2263 50  0000 C CNN
 F 2 "Connector_PinHeader_2.54mm:PinHeader_1x03_P2.54mm_Vertical" H 3400 2150 50  0001 C CNN
@@
 P 3400 2700
 AR Path="/60AC3110" Ref="JP?"  Part="1"
-AR Path="/60A8CB6A/60AC3110" Ref="JP15"  Part="1"
-F 0 "JP15" H 3400 2904 50  0000 C CNN
+AR Path="/60A8CB6A/60AC3110" Ref="JP504"  Part="1"
+F 0 "JP504" H 3400 2904 50  0000 C CNN
 F 1 "Jumper_3_Bridged12" H 3400 2813 50  0000 C CNN
 F 2 "Connector_PinHeader_2.54mm:PinHeader_1x03_P2.54mm_Vertical" H 3400 2700 50  0001 C CNN
@@
 P 3400 3250
 AR Path="/60AC311A" Ref="JP?"  Part="1"
-AR Path="/60A8CB6A/60AC311A" Ref="JP16"  Part="1"
-F 0 "JP16" H 3400 3454 50  0000 C CNN
+AR Path="/60A8CB6A/60AC311A" Ref="JP505"  Part="1"
+F 0 "JP505" H 3400 3454 50  0000 C CNN
 F 1 "Jumper_3_Bridged12" H 3400 3363 50  0000 C CNN
 F 2 "Connector_PinHeader_2.54mm:PinHeader_1x03_P2.54mm_Vertical" H 3400 3250 50  0001 C CNN
@@
 P 3400 3800
 AR Path="/60AC3124" Ref="JP?"  Part="1"
-AR Path="/60A8CB6A/60AC3124" Ref="JP17"  Part="1"
-F 0 "JP17" H 3400 4004 50  0000 C CNN
+AR Path="/60A8CB6A/60AC3124" Ref="JP506"  Part="1"
+F 0 "JP506" H 3400 4004 50  0000 C CNN
 F 1 "Jumper_3_Bridged12" H 3400 3913 50  0000 C CNN
 F 2 "Connector_PinHeader_2.54mm:PinHeader_1x03_P2.54mm_Vertical" H 3400 3800 50  0001 C CNN
@@
 P 3400 4350
 AR Path="/60AC312E" Ref="JP?"  Part="1"
-AR Path="/60A8CB6A/60AC312E" Ref="JP18"  Part="1"
-F 0 "JP18" H 3400 4554 50  0000 C CNN
+AR Path="/60A8CB6A/60AC312E" Ref="JP507"  Part="1"
+F 0 "JP507" H 3400 4554 50  0000 C CNN
 F 1 "Jumper_3_Bridged12" H 3400 4463 50  0000 C CNN
 F 2 "Connector_PinHeader_2.54mm:PinHeader_1x03_P2.54mm_Vertical" H 3400 4350 50  0001 C CNN
@@
 P 3400 5450
 AR Path="/60AC3138" Ref="JP?"  Part="1"
-AR Path="/60A8CB6A/60AC3138" Ref="JP20"  Part="1"
-F 0 "JP20" H 3400 5654 50  0000 C CNN
+AR Path="/60A8CB6A/60AC3138" Ref="JP509"  Part="1"
+F 0 "JP509" H 3400 5654 50  0000 C CNN
 F 1 "Jumper_3_Bridged12" H 3400 5563 50  0000 C CNN
 F 2 "Connector_PinHeader_2.54mm:PinHeader_1x03_P2.54mm_Vertical" H 3400 5450 50  0001 C CNN
@@
 P 3400 6000
 AR Path="/60AC3142" Ref="JP?"  Part="1"
-AR Path="/60A8CB6A/60AC3142" Ref="JP21"  Part="1"
-F 0 "JP21" H 3400 6204 50  0000 C CNN
+AR Path="/60A8CB6A/60AC3142" Ref="JP510"  Part="1"
+F 0 "JP510" H 3400 6204 50  0000 C CNN
 F 1 "Jumper_3_Bridged12" H 3400 6113 50  0000 C CNN
 F 2 "Connector_PinHeader_2.54mm:PinHeader_1x03_P2.54mm_Vertical" H 3400 6000 50  0001 C CNN
@@
 P 3400 6550
 AR Path="/60AC314C" Ref="JP?"  Part="1"
-AR Path="/60A8CB6A/60AC314C" Ref="JP23"  Part="1"
-F 0 "JP23" H 3400 6754 50  0000 C CNN
+AR Path="/60A8CB6A/60AC314C" Ref="JP511"  Part="1"
+F 0 "JP511" H 3400 6754 50  0000 C CNN
 F 1 "Jumper_3_Bridged12" H 3400 6663 50  0000 C CNN
 F 2 "Connector_PinHeader_2.54mm:PinHeader_1x03_P2.54mm_Vertical" H 3400 6550 50  0001 C CNN
@@
 P 3400 4900
 AR Path="/60AC3166" Ref="JP?"  Part="1"
-AR Path="/60A8CB6A/60AC3166" Ref="JP19"  Part="1"
-F 0 "JP19" H 3400 5104 50  0000 C CNN
+AR Path="/60A8CB6A/60AC3166" Ref="JP508"  Part="1"
+F 0 "JP508" H 3400 5104 50  0000 C CNN
 F 1 "Jumper_3_Bridged12" H 3400 5013 50  0000 C CNN
 F 2 "Connector_PinHeader_2.54mm:PinHeader_1x03_P2.54mm_Vertical" H 3400 4900 50  0001 C CNN
