File: hub75_extension/j_ds.sch (KiCad schematic (older format))
At the start: 12 parts, among them Q1 2N7002

Commit message: Yeah, just renumber the entire thing...
Parts:
- renumbered D1 to D401, JP1 to JP401, JP2 to JP402, JP3 to JP403, JP22 to JP404, JP10 to JP405, JP29 to JP406, J_DS1 to J_DS401, Q1 to Q401, R1 to R401, R2 to R402, R3 to R403
Changed lines of the file:
@@
 P 2350 3300
 AR Path="/606A0CCC" Ref="#PWR?"  Part="1"
-AR Path="/6063BB6D/606A0CCC" Ref="#PWR01"  Part="1"
-F 0 "#PWR01" H 2350 3050 50  0001 C CNN
+AR Path="/6063BB6D/606A0CCC" Ref="#PWR0403"  Part="1"
+F 0 "#PWR0403" H 2350 3050 50  0001 C CNN
 F 1 "GND" H 2355 3127 50  0000 C CNN
 F 2 "" H 2350 3300 50  0001 C CNN
@@
 P 2450 1450
 AR Path="/606A0CD9" Ref="#PWR?"  Part="1"
-AR Path="/6063BB6D/606A0CD9" Ref="#PWR02"  Part="1"
-F 0 "#PWR02" H 2450 1300 50  0001 C CNN
+AR Path="/6063BB6D/606A0CD9" Ref="#PWR0404"  Part="1"
+F 0 "#PWR0404" H 2450 1300 50  0001 C CNN
 F 1 "+3V3" H 2465 1623 50  0000 C CNN
 F 2 "" H 2450 1450 50  0001 C CNN
@@
 P 2800 2600
 AR Path="/606A0CED" Ref="JP?"  Part="1"
-AR Path="/6063BB6D/606A0CED" Ref="JP1"  Part="1"
-F 0 "JP1" H 2800 2795 50  0000 C CNN
+AR Path="/6063BB6D/606A0CED" Ref="JP401"  Part="1"
+F 0 "JP401" H 2800 2795 50  0000 C CNN
 F 1 "Jumper_2_Bridged" H 2800 2704 50  0000 C CNN
 F 2 "Connector_PinHeader_2.54mm:PinHeader_1x02_P2.54mm_Vertical" H 2800 2600 50  0001 C CNN
@@
 P 2800 2900
 AR Path="/606A0CF3" Ref="JP?"  Part="1"
-AR Path="/6063BB6D/606A0CF3" Ref="JP2"  Part="1"
-F 0 "JP2" H 2800 3095 50  0000 C CNN
+AR Path="/6063BB6D/606A0CF3" Ref="JP402"  Part="1"
+F 0 "JP402" H 2800 3095 50  0000 C CNN
 F 1 "Jumper_2_Bridged" H 2800 3004 50  0000 C CNN
 F 2 "Connector_PinHeader_2.54mm:PinHeader_1x02_P2.54mm_Vertical" H 2800 2900 50  0001 C CNN
@@
 P 2800 3300
 AR Path="/606A0CF9" Ref="JP?"  Part="1"
-AR Path="/6063BB6D/606A0CF9" Ref="JP3"  Part="1"
-F 0 "JP3" H 2800 3495 50  0000 C CNN
+AR Path="/6063BB6D/606A0CF9" Ref="JP403"  Part="1"
+F 0 "JP403" H 2800 3495 50  0000 C CNN
 F 1 "Jumper_2_Bridged" H 2800 3404 50  0000 C CNN
 F 2 "Connector_PinHeader_2.54mm:PinHeader_1x02_P2.54mm_Vertical" H 2800 3300 50  0001 C CNN
@@
 P 2800 4500
 AR Path="/606A0D0B" Ref="JP?"  Part="1"
-AR Path="/6063BB6D/606A0D0B" Ref="JP10"  Part="1"
-F 0 "JP10" H 2800 4704 50  0000 C CNN
+AR Path="/6063BB6D/606A0D0B" Ref="JP405"  Part="1"
+F 0 "JP405" H 2800 4704 50  0000 C CNN
 F 1 "Jumper_3_Bridged12" H 2800 4613 50  0000 C CNN
 F 2 "Connector_PinHeader_2.54mm:PinHeader_1x03_P2.54mm_Vertical" H 2800 4500 50  0001 C CNN
@@
 AR Path="/606A0D1E" Ref="JP?"  Part="1"
 AR Path="/602F3AD9/606A0D1E" Ref="JP?"  Part="1"
-AR Path="/6063BB6D/606A0D1E" Ref="JP22"  Part="1"
-F 0 "JP22" H 2800 4154 50  0000 C CNN
+AR Path="/6063BB6D/606A0D1E" Ref="JP404"  Part="1"
+F 0 "JP404" H 2800 4154 50  0000 C CNN
 F 1 "Jumper_3_Bridged12" H 2800 4063 50  0000 C CNN
 F 2 "Connector_PinHeader_2.54mm:PinHeader_1x03_P2.54mm_Vertical" H 2800 3950 50  0001 C CNN
@@
 P 3250 3850
 AR Path="/606CA484" Ref="#PWR?"  Part="1"
-AR Path="/6063BB6D/606CA484" Ref="#PWR040"  Part="1"
-F 0 "#PWR040" H 3250 3700 50  0001 C CNN
+AR Path="/6063BB6D/606CA484" Ref="#PWR0405"  Part="1"
+F 0 "#PWR0405" H 3250 3700 50  0001 C CNN
 F 1 "+3V3" H 3265 4023 50  0000 C CNN
 F 2 "" H 3250 3850 50  0001 C CNN
@@
 P 1400 2400
 AR Path="/606A0CC6" Ref="J_DS?"  Part="1"
-AR Path="/6063BB6D/606A0CC6" Ref="J_DS1"  Part="1"
-F 0 "J_DS1" H 1242 3565 50  0000 C CNN
+AR Path="/6063BB6D/606A0CC6" Ref="J_DS401"  Part="1"
+F 0 "J_DS401" H 1242 3565 50  0000 C CNN
 F 1 "DS_Card" H 1242 3474 50  0000 C CNN
 F 2 "ds_card_extender:IDC-Header_2x09_P2.54mm_Vertical" H 1400 2400 50  0001 C CNN
@@
 AR Path="/606EC5E7" Ref="JP?"  Part="1"
 AR Path="/602F3AD9/606EC5E7" Ref="JP?"  Part="1"
-AR Path="/6063BB6D/606EC5E7" Ref="JP29"  Part="1"
-F 0 "JP29" H 2800 5354 50  0000 C CNN
+AR Path="/6063BB6D/606EC5E7" Ref="JP406"  Part="1"
+F 0 "JP406" H 2800 5354 50  0000 C CNN
 F 1 "Jumper_3_Bridged12" H 2800 5263 50  0000 C CNN
 F 2 "Connector_PinHeader_2.54mm:PinHeader_1x03_P2.54mm_Vertical" H 2800 5150 50  0001 C CNN
@@
 RCS
 $Comp
-L Device:LED D1
+L Device:LED D401
 U 1 1 6070AB78
 P 4100 2000
-F 0 "D1" V 4139 1882 50  0000 R CNN
+F 0 "D401" V 4139 1882 50  0000 R CNN
 F 1 "LED" V 4048 1882 50  0000 R CNN
 F 2 "LED_SMD:LED_0805_2012Metric_Pad1.15x1.40mm_HandSolder" H 4100 2000 50  0001 C CNN
@@
 P 4100 1350
 AR Path="/6070AEE2" Ref="#PWR?"  Part="1"
-AR Path="/6063BB6D/6070AEE2" Ref="#PWR048"  Part="1"
-F 0 "#PWR048" H 4100 1200 50  0001 C CNN
+AR Path="/6063BB6D/6070AEE2" Ref="#PWR0408"  Part="1"
+F 0 "#PWR0408" H 4100 1200 50  0001 C CNN
 F 1 "+3V3" H 4115 1523 50  0000 C CNN
 F 2 "" H 4100 1350 50  0001 C CNN
@@
 $EndComp
 $Comp
-L Device:R R3
+L Device:R R403
 U 1 1 6070B87A
 P 4100 1600
-F 0 "R3" H 4170 1646 50  0000 L CNN
+F 0 "R403" H 4170 1646 50  0000 L CNN
 F 1 "10k" H 4170 1555 50  0000 L CNN
 F 2 "Resistor_SMD:R_0805_2012Metric_Pad1.20x1.40mm_HandSolder" V 4030 1600 50  0001 C CNN
@@
 P 4100 2250
 AR Path="/6070C342" Ref="#PWR?"  Part="1"
-AR Path="/6063BB6D/6070C342" Ref="#PWR049"  Part="1"
-F 0 "#PWR049" H 4100 2000 50  0001 C CNN
+AR Path="/6063BB6D/6070C342" Ref="#PWR0409"  Part="1"
+F 0 "#PWR0409" H 4100 2000 50  0001 C CNN
 F 1 "GND" H 4105 2077 50  0000 C CNN
 F 2 "" H 4100 2250 50  0001 C CNN
@@
 	4100 2150 4100 2250
 $Comp
-L Device:R R1
+L Device:R R401
 U 1 1 607140BA
 P 3500 4000
-F 0 "R1" H 3570 4046 50  0000 L CNN
+F 0 "R401" H 3570 4046 50  0000 L CNN
 F 1 "33k" H 3570 3955 50  0000 L CNN
 F 2 "Resistor_SMD:R_0805_2012Metric_Pad1.20x1.40mm_HandSolder" V 3430 4000 50  0001 C CNN
@@
 $EndComp
 $Comp
-L Device:R R2
+L Device:R R402
 U 1 1 60714502
 P 3500 4400
-F 0 "R2" H 3570 4446 50  0000 L CNN
+F 0 "R402" H 3570 4446 50  0000 L CNN
 F 1 "NF" H 3570 4355 50  0000 L CNN
 F 2 "Resistor_SMD:R_0805_2012Metric_Pad1.20x1.40mm_HandSolder" V 3430 4400 50  0001 C CNN
@@
 P 3500 4600
 AR Path="/60714D64" Ref="#PWR?"  Part="1"
-AR Path="/6063BB6D/60714D64" Ref="#PWR047"  Part="1"
-F 0 "#PWR047" H 3500 4350 50  0001 C CNN
+AR Path="/6063BB6D/60714D64" Ref="#PWR0407"  Part="1"
+F 0 "#PWR0407" H 3500 4350 50  0001 C CNN
 F 1 "GND" H 3505 4427 50  0000 C CNN
 F 2 "" H 3500 4600 50  0001 C CNN
@@
 $EndComp
 $Comp
-L power:+5V #PWR046
+L power:+5V #PWR0406
 U 1 1 60715408
 P 3500 3800
-F 0 "#PWR046" H 3500 3650 50  0001 C CNN
+F 0 "#PWR0406" H 3500 3650 50  0001 C CNN
 F 1 "+5V" H 3515 3973 50  0000 C CNN
 F 2 "" H 3500 3800 50  0001 C CNN
@@
 	3500 4550 3500 4600
 $Comp
-L Transistor_FET:2N7002 Q1
+L Transistor_FET:2N7002 Q401
 U 1 1 60718CEC
 P 2050 4150
-F 0 "Q1" H 2254 4196 50  0000 L CNN
+F 0 "Q401" H 2254 4196 50  0000 L CNN
 F 1 "2N7002" H 2254 4105 50  0000 L CNN
 F 2 "Package_TO_SOT_SMD:SOT-23_Handsoldering" H 2250 4075 50  0001 L CIN
@@
 P 1750 4000
 AR Path="/60722E7F" Ref="#PWR?"  Part="1"
-AR Path="/6063BB6D/60722E7F" Ref="#PWR039"  Part="1"
-F 0 "#PWR039" H 1750 3850 50  0001 C CNN
+AR Path="/6063BB6D/60722E7F" Ref="#PWR0401"  Part="1"
+F 0 "#PWR0401" H 1750 3850 50  0001 C CNN
 F 1 "+3V3" H 1765 4173 50  0000 C CNN
 F 2 "" H 1750 4000 50  0001 C CNN
@@
 P 2150 4400
 AR Path="/60724124" Ref="#PWR?"  Part="1"
-AR Path="/6063BB6D/60724124" Ref="#PWR045"  Part="1"
-F 0 "#PWR045" H 2150 4150 50  0001 C CNN
+AR Path="/6063BB6D/60724124" Ref="#PWR0402"  Part="1"
+F 0 "#PWR0402" H 2150 4150 50  0001 C CNN
 F 1 "GND" H 2155 4227 50  0000 C CNN
 F 2 "" H 2150 4400 50  0001 C CNN
