File: hub75_extension/sreg.sch (KiCad schematic (older format))
At the start: 14 parts, among them U1 74HC595, U3 NF

Commit message: Yeah, just renumber the entire thing...
Parts:
- renumbered C1 to C301, C2 to C302, JP7 to JP301, JP8 to JP302, JP9 to JP303, JP11 to JP304, JP12 to JP305, JP13 to JP306, JP14 to JP307, JP31 to JP308, JP32 to JP309, TP1 to TP301, U1 to U301, U3 to U302
Changed lines of the file:
@@
 P 2500 2300
 AR Path="/60328D52" Ref="JP?"  Part="1"
-AR Path="/602F3AD9/60328D52" Ref="JP7"  Part="1"
-F 0 "JP7" H 2500 2411 50  0000 C CNN
+AR Path="/602F3AD9/60328D52" Ref="JP301"  Part="1"
+F 0 "JP301" H 2500 2411 50  0000 C CNN
 F 1 "Jumper_3_Bridged12" H 2500 2502 50  0000 C CNN
 F 2 "Connector_PinHeader_2.54mm:PinHeader_1x03_P2.54mm_Vertical" H 2500 2300 50  0001 C CNN
@@
 P 2500 2850
 AR Path="/60328D58" Ref="JP?"  Part="1"
-AR Path="/602F3AD9/60328D58" Ref="JP8"  Part="1"
-F 0 "JP8" H 2500 3054 50  0000 C CNN
+AR Path="/602F3AD9/60328D58" Ref="JP302"  Part="1"
+F 0 "JP302" H 2500 3054 50  0000 C CNN
 F 1 "Jumper_3_Bridged12" H 2500 2963 50  0000 C CNN
 F 2 "Connector_PinHeader_2.54mm:PinHeader_1x03_P2.54mm_Vertical" H 2500 2850 50  0001 C CNN
@@
 P 2150 2100
 AR Path="/60328D5E" Ref="#PWR?"  Part="1"
-AR Path="/602F3AD9/60328D5E" Ref="#PWR031"  Part="1"
-F 0 "#PWR031" H 2150 1950 50  0001 C CNN
+AR Path="/602F3AD9/60328D5E" Ref="#PWR0303"  Part="1"
+F 0 "#PWR0303" H 2150 1950 50  0001 C CNN
 F 1 "+3V3" H 2165 2273 50  0000 C CNN
 F 2 "" H 2150 2100 50  0001 C CNN
@@
 P 2500 2100
 AR Path="/60328D66" Ref="#PWR?"  Part="1"
-AR Path="/602F3AD9/60328D66" Ref="#PWR033"  Part="1"
-F 0 "#PWR033" H 2500 1950 50  0001 C CNN
+AR Path="/602F3AD9/60328D66" Ref="#PWR0305"  Part="1"
+F 0 "#PWR0305" H 2500 1950 50  0001 C CNN
 F 1 "VCC" H 2515 2273 50  0000 C CNN
 F 2 "" H 2500 2100 50  0001 C CNN
@@
 P 2850 2100
 AR Path="/60328D6C" Ref="#PWR?"  Part="1"
-AR Path="/602F3AD9/60328D6C" Ref="#PWR034"  Part="1"
-F 0 "#PWR034" H 2850 1950 50  0001 C CNN
+AR Path="/602F3AD9/60328D6C" Ref="#PWR0306"  Part="1"
+F 0 "#PWR0306" H 2850 1950 50  0001 C CNN
 F 1 "+5V" H 2865 2273 50  0000 C CNN
 F 2 "" H 2850 2100 50  0001 C CNN
@@
 P 2950 2750
 AR Path="/60328D75" Ref="#PWR?"  Part="1"
-AR Path="/602F3AD9/60328D75" Ref="#PWR035"  Part="1"
-F 0 "#PWR035" H 2950 2600 50  0001 C CNN
+AR Path="/602F3AD9/60328D75" Ref="#PWR0307"  Part="1"
+F 0 "#PWR0307" H 2950 2600 50  0001 C CNN
 F 1 "VCC" H 2965 2923 50  0000 C CNN
 F 2 "" H 2950 2750 50  0001 C CNN
@@
 P 2150 3000
 AR Path="/60328D7B" Ref="#PWR?"  Part="1"
-AR Path="/602F3AD9/60328D7B" Ref="#PWR032"  Part="1"
-F 0 "#PWR032" H 2150 2750 50  0001 C CNN
+AR Path="/602F3AD9/60328D7B" Ref="#PWR0304"  Part="1"
+F 0 "#PWR0304" H 2150 2750 50  0001 C CNN
 F 1 "GND" H 2155 2827 50  0000 C CNN
 F 2 "" H 2150 3000 50  0001 C CNN
@@
 P 4200 2000
 AR Path="/60328D8B" Ref="#PWR?"  Part="1"
-AR Path="/602F3AD9/60328D8B" Ref="#PWR037"  Part="1"
-F 0 "#PWR037" H 4200 1850 50  0001 C CNN
+AR Path="/602F3AD9/60328D8B" Ref="#PWR0311"  Part="1"
+F 0 "#PWR0311" H 4200 1850 50  0001 C CNN
 F 1 "VCC" H 4215 2173 50  0000 C CNN
 F 2 "" H 4200 2000 50  0001 C CNN
@@
 P 5650 2500
 AR Path="/60328D98" Ref="JP?"  Part="1"
-AR Path="/602F3AD9/60328D98" Ref="JP11"  Part="1"
-F 0 "JP11" H 5650 2695 50  0000 C CNN
+AR Path="/602F3AD9/60328D98" Ref="JP304"  Part="1"
+F 0 "JP304" H 5650 2695 50  0000 C CNN
 F 1 "Jumper_2_Bridged" H 5650 2604 50  0000 C CNN
 F 2 "Connector_PinHeader_2.54mm:PinHeader_1x02_P2.54mm_Vertical" H 5650 2500 50  0001 C CNN
@@
 P 5650 2800
 AR Path="/60328DA0" Ref="JP?"  Part="1"
-AR Path="/602F3AD9/60328DA0" Ref="JP12"  Part="1"
-F 0 "JP12" H 5650 2995 50  0000 C CNN
+AR Path="/602F3AD9/60328DA0" Ref="JP305"  Part="1"
+F 0 "JP305" H 5650 2995 50  0000 C CNN
 F 1 "Jumper_2_Bridged" H 5650 2904 50  0000 C CNN
 F 2 "Connector_PinHeader_2.54mm:PinHeader_1x02_P2.54mm_Vertical" H 5650 2800 50  0001 C CNN
@@
 P 5650 3100
 AR Path="/60328DA6" Ref="JP?"  Part="1"
-AR Path="/602F3AD9/60328DA6" Ref="JP13"  Part="1"
-F 0 "JP13" H 5650 3295 50  0000 C CNN
+AR Path="/602F3AD9/60328DA6" Ref="JP306"  Part="1"
+F 0 "JP306" H 5650 3295 50  0000 C CNN
 F 1 "Jumper_2_Bridged" H 5650 3204 50  0000 C CNN
 F 2 "Connector_PinHeader_2.54mm:PinHeader_1x02_P2.54mm_Vertical" H 5650 3100 50  0001 C CNN
@@
 P 5650 3400
 AR Path="/60328DAC" Ref="JP?"  Part="1"
-AR Path="/602F3AD9/60328DAC" Ref="JP14"  Part="1"
-F 0 "JP14" H 5650 3595 50  0000 C CNN
+AR Path="/602F3AD9/60328DAC" Ref="JP307"  Part="1"
+F 0 "JP307" H 5650 3595 50  0000 C CNN
 F 1 "Jumper_2_Bridged" H 5650 3504 50  0000 C CNN
 F 2 "Connector_PinHeader_2.54mm:PinHeader_1x02_P2.54mm_Vertical" H 5650 3400 50  0001 C CNN
@@
 P 4200 3700
 AR Path="/60328DC5" Ref="#PWR?"  Part="1"
-AR Path="/602F3AD9/60328DC5" Ref="#PWR038"  Part="1"
-F 0 "#PWR038" H 4200 3450 50  0001 C CNN
+AR Path="/602F3AD9/60328DC5" Ref="#PWR0312"  Part="1"
+F 0 "#PWR0312" H 4200 3450 50  0001 C CNN
 F 1 "GND" H 4205 3527 50  0000 C CNN
 F 2 "" H 4200 3700 50  0001 C CNN
@@
 P 1800 2600
 AR Path="/60328DCD" Ref="C?"  Part="1"
-AR Path="/602F3AD9/60328DCD" Ref="C1"  Part="1"
-F 0 "C1" H 1915 2646 50  0000 L CNN
+AR Path="/602F3AD9/60328DCD" Ref="C301"  Part="1"
+F 0 "C301" H 1915 2646 50  0000 L CNN
 F 1 "100n" H 1915 2555 50  0000 L CNN
 F 2 "Capacitor_SMD:C_0805_2012Metric_Pad1.18x1.45mm_HandSolder" H 1838 2450 50  0001 C CNN
@@
 P 1800 2450
 AR Path="/60328DD3" Ref="#PWR?"  Part="1"
-AR Path="/602F3AD9/60328DD3" Ref="#PWR08"  Part="1"
-F 0 "#PWR08" H 1800 2300 50  0001 C CNN
+AR Path="/602F3AD9/60328DD3" Ref="#PWR0301"  Part="1"
+F 0 "#PWR0301" H 1800 2300 50  0001 C CNN
 F 1 "VCC" H 1815 2623 50  0000 C CNN
 F 2 "" H 1800 2450 50  0001 C CNN
@@
 P 1800 2750
 AR Path="/60328DD9" Ref="#PWR?"  Part="1"
-AR Path="/602F3AD9/60328DD9" Ref="#PWR030"  Part="1"
-F 0 "#PWR030" H 1800 2500 50  0001 C CNN
+AR Path="/602F3AD9/60328DD9" Ref="#PWR0302"  Part="1"
+F 0 "#PWR0302" H 1800 2500 50  0001 C CNN
 F 1 "GND" H 1805 2577 50  0000 C CNN
 F 2 "" H 1800 2750 50  0001 C CNN
@@
 P 4850 4100
 AR Path="/60328DDF" Ref="TP?"  Part="1"
-AR Path="/602F3AD9/60328DDF" Ref="TP1"  Part="1"
-F 0 "TP1" V 4804 4288 50  0000 L CNN
+AR Path="/602F3AD9/60328DDF" Ref="TP301"  Part="1"
+F 0 "TP301" V 4804 4288 50  0000 L CNN
 F 1 "TestPoint" V 4895 4288 50  0000 L CNN
 F 2 "Connector_PinHeader_2.54mm:PinHeader_1x01_P2.54mm_Vertical" H 5050 4100 50  0001 C CNN
@@
 P 3450 2200
 AR Path="/60328DE5" Ref="JP?"  Part="1"
-AR Path="/602F3AD9/60328DE5" Ref="JP9"  Part="1"
-F 0 "JP9" H 3450 2404 50  0000 C CNN
+AR Path="/602F3AD9/60328DE5" Ref="JP303"  Part="1"
+F 0 "JP303" H 3450 2404 50  0000 C CNN
 F 1 "Jumper_3_Bridged12" H 3450 2313 50  0000 C CNN
 F 2 "Connector_PinHeader_2.54mm:PinHeader_1x03_P2.54mm_Vertical" H 3450 2200 50  0001 C CNN
@@
 P 3250 2650
 AR Path="/60328DF1" Ref="#PWR?"  Part="1"
-AR Path="/602F3AD9/60328DF1" Ref="#PWR036"  Part="1"
-F 0 "#PWR036" H 3250 2500 50  0001 C CNN
+AR Path="/602F3AD9/60328DF1" Ref="#PWR0310"  Part="1"
+F 0 "#PWR0310" H 3250 2500 50  0001 C CNN
 F 1 "VCC" H 3265 2823 50  0000 C CNN
 F 2 "" H 3250 2650 50  0001 C CNN
@@
 P 3200 5000
 AR Path="/60842BC8" Ref="C?"  Part="1"
-AR Path="/602F3AD9/60842BC8" Ref="C2"  Part="1"
-F 0 "C2" H 3315 5046 50  0000 L CNN
+AR Path="/602F3AD9/60842BC8" Ref="C302"  Part="1"
+F 0 "C302" H 3315 5046 50  0000 L CNN
 F 1 "100n" H 3315 4955 50  0000 L CNN
 F 2 "Capacitor_SMD:C_0805_2012Metric_Pad1.18x1.45mm_HandSolder" H 3238 4850 50  0001 C CNN
@@
 P 3200 4850
 AR Path="/60842BCE" Ref="#PWR?"  Part="1"
-AR Path="/602F3AD9/60842BCE" Ref="#PWR052"  Part="1"
-F 0 "#PWR052" H 3200 4700 50  0001 C CNN
+AR Path="/602F3AD9/60842BCE" Ref="#PWR0308"  Part="1"
+F 0 "#PWR0308" H 3200 4700 50  0001 C CNN
 F 1 "VCC" H 3215 5023 50  0000 C CNN
 F 2 "" H 3200 4850 50  0001 C CNN
@@
 P 3200 5150
 AR Path="/60842BD4" Ref="#PWR?"  Part="1"
-AR Path="/602F3AD9/60842BD4" Ref="#PWR053"  Part="1"
-F 0 "#PWR053" H 3200 4900 50  0001 C CNN
+AR Path="/602F3AD9/60842BD4" Ref="#PWR0309"  Part="1"
+F 0 "#PWR0309" H 3200 4900 50  0001 C CNN
 F 1 "GND" H 3205 4977 50  0000 C CNN
 F 2 "" H 3200 5150 50  0001 C CNN
@@
 P 4200 5350
 AR Path="/60847B05" Ref="U?"  Part="1"
-AR Path="/602F3AD9/60847B05" Ref="U3"  Part="1"
-F 0 "U3" H 4200 6131 50  0000 C CNN
+AR Path="/602F3AD9/60847B05" Ref="U302"  Part="1"
+F 0 "U302" H 4200 6131 50  0000 C CNN
 F 1 "NF" H 4200 6040 50  0000 C CNN
 F 2 "Package_SO:SOIC-16_3.9x9.9mm_P1.27mm" H 4200 5350 50  0001 C CNN
@@
 P 4200 4450
 AR Path="/60847B0B" Ref="#PWR?"  Part="1"
-AR Path="/602F3AD9/60847B0B" Ref="#PWR054"  Part="1"
-F 0 "#PWR054" H 4200 4300 50  0001 C CNN
+AR Path="/602F3AD9/60847B0B" Ref="#PWR0313"  Part="1"
+F 0 "#PWR0313" H 4200 4300 50  0001 C CNN
 F 1 "VCC" H 4215 4623 50  0000 C CNN
 F 2 "" H 4200 4450 50  0001 C CNN
@@
 P 4200 6150
 AR Path="/60847B12" Ref="#PWR?"  Part="1"
-AR Path="/602F3AD9/60847B12" Ref="#PWR055"  Part="1"
-F 0 "#PWR055" H 4200 5900 50  0001 C CNN
+AR Path="/602F3AD9/60847B12" Ref="#PWR0314"  Part="1"
+F 0 "#PWR0314" H 4200 5900 50  0001 C CNN
 F 1 "GND" H 4205 5977 50  0000 C CNN
 F 2 "" H 4200 6150 50  0001 C CNN
@@
 P 5650 3650
 AR Path="/609589F5" Ref="JP?"  Part="1"
-AR Path="/602F3AD9/609589F5" Ref="JP31"  Part="1"
-F 0 "JP31" H 5650 3845 50  0000 C CNN
+AR Path="/602F3AD9/609589F5" Ref="JP308"  Part="1"
+F 0 "JP308" H 5650 3845 50  0000 C CNN
 F 1 "Jumper_2_Bridged" H 5650 3754 50  0000 C CNN
 F 2 "Connector_PinHeader_2.54mm:PinHeader_1x02_P2.54mm_Vertical" H 5650 3650 50  0001 C CNN
@@
 P 5650 3900
 AR Path="/609A10D5" Ref="JP?"  Part="1"
-AR Path="/602F3AD9/609A10D5" Ref="JP32"  Part="1"
-F 0 "JP32" H 5650 4095 50  0000 C CNN
+AR Path="/602F3AD9/609A10D5" Ref="JP309"  Part="1"
+F 0 "JP309" H 5650 4095 50  0000 C CNN
 F 1 "Jumper_2_Bridged" H 5650 4004 50  0000 C CNN
 F 2 "Connector_PinHeader_2.54mm:PinHeader_1x02_P2.54mm_Vertical" H 5650 3900 50  0001 C CNN
@@
 P 4200 2900
 AR Path="/60328D4C" Ref="U?"  Part="1"
-AR Path="/602F3AD9/60328D4C" Ref="U1"  Part="1"
-F 0 "U1" H 4200 3681 50  0000 C CNN
+AR Path="/602F3AD9/60328D4C" Ref="U301"  Part="1"
+F 0 "U301" H 4200 3681 50  0000 C CNN
 F 1 "74HC595" H 4200 3590 50  0000 C CNN
 F 2 "Package_SO:SOIC-16_3.9x9.9mm_P1.27mm" H 4200 2900 50  0001 C CNN
